File: Eagle_Board_Files/MP26123_4/MPS_Charge_Controller.brd (EAGLE design)
At the start: 62 x 54 mm, 48 parts, among them IC1 FDS4435BZ, IC2 MP26123DR-LF-Z, IC3 FDS4435BZ, IC4 74132D, J1 VIN, J2 NTC Sensor, J3 Pi Signals, J4 Power Control, J5 Power Supply Loads, J6 Battery Connections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

Commit message: Add files via upload
Parts:
- C6: value 0.1µF -> 0.15µF
Changed lines of the file:
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@@
 <attribute name="VALUE" x="30.59" y="26.261" size="0.6096" layer="27" font="vector" ratio="20" align="top-center"/>
 </element>
-<element name="C6" library="SparkFun-Capacitors" package="0805" value="0.1µF" x="33.5" y="27.85" smashed="yes" rot="R90">
+<element name="C6" library="SparkFun-Capacitors" package="0805" value="0.15µF" x="33.5" y="27.85" smashed="yes" rot="R90">
 <attribute name="NAME" x="32.611" y="27.85" size="0.6096" layer="25" font="vector" ratio="20" rot="R90" align="bottom-center"/>
 <attribute name="PROD_ID" value="CAP-08469" x="66.52" y="65.95" size="1.778" layer="27" rot="R90" display="off"/>

Commit message: Add files via upload
Parts:
- removed R3: OPEN, 0603_RESISTOR:0603_RESISTOR
- added C17: 2.2µF, SparkFun-Capacitors:0805
- added J9: 3.3V AP, SparkFun-Connectors:1X02
- added U1: AP7381-33Y-13, AP7381:AP7381
- J7: value 3.3V TP -> 3.3V MP
- moved R7 18.5 mm to (7.81, 12.5)
- moved R4 13.3 mm to (23.9, 18.7)
- moved C13 5.37 mm to (12.5, 15.2), turned to 270 degrees
- moved R1 3.24 mm to (7.85, 16.5), turned to 270 degrees
- moved R2 2.86 mm to (7.80, 21.6)
- moved J5 0.16 mm to (4.79, 47.4)
- moved J8 0.10 mm to (26.6, 5.69)
Connections:
- new net MP3V3: C4.1, IC2.5, J7.1, R4.2, R9.2
- net FUSE_OUT: no longer R3.1
- net GND: now also C17.2, J9.1, U1.P$3, U1.P$4; no longer R3.2
- net V3P3: now also C17.1, J9.2, U1.P$1; no longer C4.1, IC2.5, J7.1, R4.2, R9.2
- net VLOAD: now also U1.P$2
Routing:
- net MP3V3: track 0.00 -> 27.8 mm
- net V3P3: track 53.3 -> 25.5 mm
- net VLOAD: track 273.6 -> 285.3 mm, vias 0 -> 2
- net NTC: track 28.0 -> 32.9 mm, vias 0 -> 1
- net GND: track 59.8 -> 62.8 mm, vias 98 -> 99
- net DISABLE: track 32.7 -> 30.4 mm
- net FUSE_OUT: track 15.4 -> 13.6 mm
- net CHGOK: track 33.3 -> 35.0 mm
Other:
- board text added: "3.3VAP"
- board text added: "3.3VMP"
- board text added: "CHGOK"
- board text added: "Disable"
- board text added: "En"
- board text added: "PS_EN"
- board text added: "PS_En"
- board text added: "Rev 1.1"
- board text added: "SR_Off"
- board text added: "SR_On"
- board text removed: "3.3V"
- board text removed: "CHRG_Off"
- board text removed: "En*"
- board text removed: "OK"
- board text removed: "PS_EN*"
- board text removed: "PS_En*"
- board text removed: "RS_Off"
- board text removed: "RS_On"
