File: Eagle_Board_Files/MP26123_4/MPS_Charge_Controller.sch (EAGLE design)
At the start: 47 parts, among them IC1 FDS4435BZ, IC2 MP26123DR-LF-Z, IC3 FDS4435BZ, IC4 74132D, J1 VIN, J2 NTC Sensor, J3 Pi Signals, J4 Power Control, J5 Power Supply Loads, J6 Battery Connections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

Commit message: Add files via upload
Parts:
- C6: value 0.1µF -> 0.15µF
Changed lines of the file:
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@@
 <part name="C3" library="SparkFun-Capacitors" deviceset="0.33UF/330NF" device="-0805-50V-10%" value="0.1µF"/>
 <part name="C2" library="SparkFun-Capacitors" deviceset="0.33UF/330NF" device="-0805-50V-10%" value="0.1µF"/>
-<part name="C6" library="SparkFun-Capacitors" deviceset="0.33UF/330NF" device="-0805-50V-10%" value="0.1µF"/>
+<part name="C6" library="SparkFun-Capacitors" deviceset="0.33UF/330NF" device="-0805-50V-10%" value="0.15µF"/>
 <part name="GND9" library="SparkFun-PowerSymbols" deviceset="GND" device=""/>
 <part name="R11" library="0603_RESISTOR" deviceset="0603_RESISTOR" device="" value="750"/>

Commit message: Add files via upload
Parts:
- removed R3: OPEN, 0603_RESISTOR:0603_RESISTOR
- added C17: 2.2µF, SparkFun-Capacitors:0.33UF/330NF-0805-50V-10%
- added J9: 3.3V AP, SparkFun-Connectors:CONN_02
- added U1: AP7381-33Y-13, AP7381:AP7381
- J7: value 3.3V TP -> 3.3V MP
Connections:
- new net MP3V3: C4.1, IC2.VREF33, J7.1, R4.2, R9.2
- net FUSE_OUT: no longer R3.1
- net GND: now also C17.2, J9.1, U1.GND; no longer R3.2
- net V3P3: now also C17.1, J9.2, U1.VOUT; no longer C4.1, IC2.VREF33, J7.1, R4.2, R9.2
- net VLOAD: now also U1.VIN
Other:
- moved on the sheet: J7, L1
